File: kicad/Design_Elec.kicad_pcb (KiCad board)
At the start: 2 copper layers, 32 x 22 mm, 17 parts, among them J3 FDTI, SW1 SW_Push, U1 ATmega328P-A

Commit message: Lulumix
Parts:
- added L: LOGO, FootPrint:LuluMix, F.Cu at (80.0, 96.8)
- C1, C2: moved to F.Cu
- moved C4 46.2 mm to (52.9, 91.7), turned to 90 degrees
- moved R3 40.6 mm to (58.9, 91.4), turned to -90 degrees
- moved SW1 40.4 mm to (55.9, 91.9), turned to 0 degrees
- moved C6 38.1 mm to (51.2, 89.4)
- moved C3 38.0 mm to (75.0, 93.0), turned to 135 degrees
- moved C7 35.9 mm to (53.3, 96.2), turned to 90 degrees
- moved U1 35.9 mm to (70.5, 96.5), turned to 45 degrees
- moved J3 35.8 mm to (50.9, 97.6)
- moved D1 35.6 mm to (58.7, 93.7), turned to 0 degrees
- moved C1 35.4 mm to (61.4, 101.4)
- moved C2 35.4 mm to (61.6, 98.1)
- moved D2 34.9 mm to (55.1, 97.7), turned to 180 degrees
- moved Y1 34.8 mm to (63.2, 99.7)
- moved R2 33.9 mm to (54.8, 96.0)
- moved J1 33.4 mm to (67.7, 103.9)
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Connections:
- U1 pad 21: (no net) -> unconnected-(U1-Pad21)
- U1 pad 5: (no net) -> unconnected-(U1-Pad5)
- U1 pad 6: (no net) -> unconnected-(U1-Pad6)
Routing:
- net SCK: track 39.3 -> 22.4 mm
- net MISO: track 18.2 -> 9.37 mm
- net A1: track 11.8 -> 3.64 mm
- net A0: track 11.4 -> 3.36 mm
- net A2: track 11.9 -> 4.07 mm
- net MOSI: track 19.4 -> 11.8 mm
- net D2: track 16.7 -> 9.14 mm, vias 0 -> 1
- net A3: track 13.6 -> 6.11 mm
- net TXO: track 27.1 -> 20.2 mm
- net D10: track 20.8 -> 14.0 mm
- net D3: track 13.2 -> 6.47 mm, vias 0 -> 1
- net RXI: track 30.3 -> 25.3 mm, vias 0 -> 1
- net D4: track 11.9 -> 7.02 mm, vias 0 -> 1
- net Net-(U1-XTAL1/PB6): track 5.20 -> 8.89 mm, vias 2 -> 0
- net D5: track 5.16 -> 2.43 mm
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Other:
- board size 32 x 22 mm -> 33.6 x 17.7 mm
