File: kicad/Design_Elec.kicad_pcb (KiCad board)
At the start: 2 copper layers, 33.6 x 17.7 mm, 18 parts, among them J3 FDTI, SW1 SW_Push, U1 ATmega328P-A

Commit message: Done ig
Parts:
- moved D1 1.15 mm to (58.5, 94.8)
- moved C1 1.15 mm to (60.2, 101.4)
- moved Y1 0.80 mm to (62.5, 100.0)
- moved C2 0.80 mm to (60.9, 98.4)
- moved R1 0.61 mm to (60.3, 93.5)
Routing:
- net GND: track 45.2 -> 42.3 mm
- net D2: track 9.14 -> 10.7 mm
- net Net-(U1-XTAL1/PB6): track 8.89 -> 7.71 mm
- net D3: track 6.47 -> 7.51 mm
- net SCK: track 22.4 -> 23.1 mm
- net RXI: track 25.3 -> 25.9 mm
- net D4: track 7.02 -> 7.65 mm
- net Net-(D1-Pad2): track 0.89 -> 1.51 mm
