File: kicad/Design_Elec.kicad_sch (KiCad schematic)
At the start: 17 parts, among them J3 FDTI, SW1 SW_Push, U1 ATmega328P-A

Commit message: Need to l;ink the thing
Parts:
- removed U1: ATmega328P-A, symbol Symbol_lib:ATmega328P-A
- added U1: ATmega328P-A, FootPrint:ATmega328P-AB-TQFP-32_7x7x1.2mm_P0.8mm, symbol Symbol_lib:ATmega328P-AB
Connections:
- net A0: now also U1.23 (PC0)
- net A1: now also U1.24 (PC1)
- net A2: now also U1.25 (PC2)
- net A3: now also U1.26 (PC3)
- net A4: now also U1.27 (PC4)
- net A5: now also U1.28 (PC5)
- net A6: now also U1.19 (ADC6)
- net A7: now also U1.22 (ADC7)
- net D10: now also U1.14 (PB2)
- net D2: now also U1.32 (PD2)
- net D3: now also U1.1 (PD3)
- net D4: now also U1.2 (PD4)
- net D5: now also U1.9 (PD5)
- net D6: now also U1.10 (PD6)
- net D7: now also U1.11 (PD7)
- net D8: now also U1.12 (PB0)
- net D9: now also U1.13 (PB1)
- net DTR: now also U1.29 (RESET/PC6)
- net GND: now also U1.3 (GND)
- net MISO: now also U1.16 (PB4)
- net MOSI: now also U1.15 (PB3)
- net RXI: now also U1.30 (PD0)
- net SCK: now also U1.17 (PB5)
- net TXO: now also U1.31 (PD1)
- net VCC: now also U1.18 (AVCC), U1.4 (VCC)
- net at C1.1, Y1.3: now also U1.8 (XTAL2/PB7)
- net at C3.2: now also U1.20 (AREF)
- net at C2.1, Y1.1: now also U1.7 (XTAL1/PB6)
Other:
- moved on the sheet: D1, D2

Commit message: PCB SWAG
Parts:
- C1, C2, C3, C4, C6, C7: footprint (none) -> FootPrint:C0603-DA-DimCode_1.7x0.9x0.9mm_P0.4mm
- D1, D2: footprint (none) -> FootPrint:LED-0603_1.6x0.8x0.6mm_P1.2mm
- J1, J2: footprint (none) -> FootPrint:PinHeader-1x12_30.3x2.5x8.5mm_T3mm_P2.54mm
- J3: footprint (none) -> FootPrint:PinHeader-1x06_15.05x2.5x8.5mm_T3mm_P2.54mm
- R1, R2, R3: footprint (none) -> FootPrint:R0603_1.75x0.95x0.55mm_P1.3mm
- SW1: footprint (none) -> FootPrint:SW-B3U-1000P_4x2.5x1.7mm_P2.65mm
- Y1: footprint (none) -> FootPrint:Crystal-YSX321SL_3.2x2.5x0.7mm
Changed lines of the file:
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@@
 			)
 		)
-		(property "Footprint" ""
+		(property "Footprint" "FootPrint:R0603_1.75x0.95x0.55mm_P1.3mm"
 			(at 109.22 38.1 0)
 			(effects
@@
 			)
 		)
-		(property "Footprint" ""
+		(property "Footprint" "FootPrint:C0603-DA-DimCode_1.7x0.9x0.9mm_P0.4mm"
 			(at 151.765 45.72 0)
 			(effects
@@
 			)
 		)
-		(property "Footprint" ""
+		(property "Footprint" "FootPrint:C0603-DA-DimCode_1.7x0.9x0.9mm_P0.4mm"
 			(at 127.635 123.19 0)
 			(effects
@@
 			)
 		)
-		(property "Footprint" ""
+		(property "Footprint" "FootPrint:C0603-DA-DimCode_1.7x0.9x0.9mm_P0.4mm"
 			(at 60.325 96.52 0)
 			(effects
@@
 			)
 		)
-		(property "Footprint" ""
+		(property "Footprint" "FootPrint:C0603-DA-DimCode_1.7x0.9x0.9mm_P0.4mm"
 			(at 54.61 46.355 0)
 			(effects
@@
 			)
 		)
-		(property "Footprint" ""
+		(property "Footprint" "FootPrint:C0603-DA-DimCode_1.7x0.9x0.9mm_P0.4mm"
 			(at 127.635 111.76 0)
 			(effects
@@
 			)
 		)
-		(property "Footprint" ""
+		(property "Footprint" "FootPrint:R0603_1.75x0.95x0.55mm_P1.3mm"
 			(at 67.31 49.53 0)
 			(effects
@@
 			)
 		)
-		(property "Footprint" ""
+		(property "Footprint" "FootPrint:C0603-DA-DimCode_1.7x0.9x0.9mm_P0.4mm"
 			(at 45.72 46.355 0)
 			(effects
@@
 			)
 		)
-		(property "Footprint" ""
+		(property "Footprint" "FootPrint:Crystal-YSX321SL_3.2x2.5x0.7mm"
 			(at 120.65 116.205 0)
 			(effects
@@
 			)
 		)
-		(property "Footprint" ""
+		(property "Footprint" "FootPrint:LED-0603_1.6x0.8x0.6mm_P1.2mm"
 			(at 39.37 81.28 0)
 			(effects
@@
 			)
 		)
-		(property "Footprint" ""
+		(property "Footprint" "FootPrint:PinHeader-1x06_15.05x2.5x8.5mm_T3mm_P2.54mm"
 			(at -25.4 426.72 0)
 			(effects
@@
 			)
 		)
-		(property "Footprint" ""
+		(property "Footprint" "FootPrint:LED-0603_1.6x0.8x0.6mm_P1.2mm"
 			(at 81.28 82.55 0)
 			(effects
@@
 			)
 		)
-		(property "Footprint" ""
+		(property "Footprint" "FootPrint:SW-B3U-1000P_4x2.5x1.7mm_P2.65mm"
 			(at 158.75 45.72 0)
 			(effects
@@
 			)
 		)
-		(property "Footprint" ""
+		(property "Footprint" "FootPrint:R0603_1.75x0.95x0.55mm_P1.3mm"
 			(at 166.37 41.91 0)
 			(effects
@@
 			)
 		)
-		(property "Footprint" ""
+		(property "Footprint" "FootPrint:PinHeader-1x12_30.3x2.5x8.5mm_T3mm_P2.54mm"
 			(at 453.39 -210.82 0)
 			(effects
@@
 			)
 		)
-		(property "Footprint" ""
+		(property "Footprint" "FootPrint:PinHeader-1x12_30.3x2.5x8.5mm_T3mm_P2.54mm"
 			(at -85.09 429.26 0)
 			(effects

Commit message: Lulumix
Changed lines of the file:
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@@
 		(pin "13"
+		)
+		(pin "21"
+		)
+		(pin "5"
+		)
+		(pin "6"
 		)
 		(instances
