File: kicad/Final_6.5x12_0via_Teardrop_GND-Plane.kicad_pcb.kicad_pcb (KiCad board)
At the start: 2 copper layers, 33.6 x 17.7 mm, 18 parts, among them J3 FDTI, SW1 SW_Push, U1 ATmega328P-A

Commit message: a
Routing:
- net GND: track 83.9 -> 69.5 mm
- added copper zone on B.Cu, net GND

Commit message: ew
Routing:
- net GND: track 69.5 -> 18.8 mm, vias 0 -> 3
- net DTR: track 41.1 -> 30.7 mm
- net TXO: track 22.7 -> 14.7 mm
- net RAW: track 61.0 -> 53.7 mm
- added copper zone on F.Cu, net DTR
- added copper zone on F.Cu, net GND
- added copper zone on F.Cu, net RAW
- added copper zone on F.Cu, net TXO

Commit message: a
Routing:
- net RAW: track 53.7 -> 50.7 mm
- net SCK: track 8.58 -> 9.55 mm
- net A2: track 4.07 -> 4.98 mm
